File: pcb/ae-temp-monitor.kicad_sch (KiCad schematic)
At the start: 25 parts, among them J1 USB_C_Receptacle_USB2.0, Q1 AP3415E, SW1 SW_Push, SW2 SW_Push, U1 ESP32-C3-MINI-1, U2 TMP102xxDRL, U4 AP2112K-3.3

Commit message: working
Other:
- note added: "Need to shut down LDO when on Batt"
Changed lines of the file:
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@@
+		)
+	)
+	(text "Need to shut down LDO when on Batt"
+		(exclude_from_sim no)
+		(at 98.552 157.226 0)
+		(effects
+			(font
+				(size 2.032 2.032)
+				(color 255 62 71 1)
+			)
+			(justify left bottom)
 		)
 	)
